Commit message: Fixed robot frame and code in ball_chaser and launch file

File: my_robot/urdf/my_robot.xacro (robot description, xacro)
@@ -25,5 +25,5 @@
   <link name="robot_footprint"></link>
   <joint name="robot_footprint_joint" type="fixed">
-    <origin xyz="-2.43 -2.49 0.3" rpy="0 0 0" />
+    <origin xyz="-2.43 -2.49 0.0" rpy="0 0 0" />
     <parent link="robot_footprint"/>
     <child link="chassis" />
@@ -34,5 +34,5 @@
     <inertial>
       <mass value="15.0"/>
-      <origin xyz="0.0 0 0.2" rpy=" 0 0 0"/>
+      <origin xyz="0 0 0" rpy=" 0 0 0"/>
       <inertia
           ixx="0.1" ixy="0" ixz="0"
